Commit message: updated frame names

File: urdf/fp3_1.urdf (robot description, URDF)
Before this commit: robot fp3_1, 14 links, 13 joints
Links:
- removed link base
- added link fp3_1_base
Joints:
- joint fp3_1_base_joint: parent base -> fp3_1_base

File: urdf/fp3_2.urdf (robot description, URDF)
Before this commit: robot fp3_2, 14 links, 13 joints
Links:
- removed link base
- added link fp3_2_base
Joints:
- joint fp3_2_base_joint: parent base -> fp3_2_base
